Commit message: inspector motion library, move on circle, move around point, sensor orientation

File: urdf/robotic_arm_inspector.urdf.xacro (robot description, xacro)
@@ -8,8 +8,14 @@
   <!-- <xacro:include filename="$(find common_sensors)/urdf/sensors/kinect2.urdf.xacro" /> -->
   <link name="world" />
-  <joint name="base_arm" type="fixed">
+  <joint name="world_joint" type="fixed">
     <parent link="world" />
+    <child link = "cart" />
+    <origin xyz="0.0 0.0 1.0" rpy="0.0 0.0 0.0" />
+  </joint>
+  <link name = "cart"/>
+  <joint name="cart_joint" type="fixed">
+    <parent link="cart" />
     <child link = "base_link" />
-    <origin xyz="0.0 0.0 0.0" rpy="0.0 0.0 0.0" />
+    <origin xyz="0.0 0.5 0.25" rpy="1.570796 0.0 1.570796" />
   </joint>
   <xacro:ur5_robot prefix="" joint_limited="true"

Commit message: motion lib & train inspactor lib

File: urdf/robotic_arm_inspector.urdf.xacro (robot description, xacro)
@@ -17,5 +17,5 @@
     <parent link="cart" />
     <child link = "base_link" />
-    <origin xyz="0.0 0.5 0.25" rpy="1.570796 0.0 1.570796" />
+    <origin xyz="0.0 1.6 0.25" rpy="1.570796 0.0 1.570796" />
   </joint>
   <xacro:ur5_robot prefix="" joint_limited="true"

Commit message: fixing models

File: urdf/robotic_arm_inspector.urdf.xacro (robot description, xacro)
@@ -17,5 +17,5 @@
     <parent link="cart" />
     <child link = "base_link" />
-    <origin xyz="0.0 1.6 0.25" rpy="1.570796 0.0 1.570796" />
+    <origin xyz="0.0 0.7 0.0" rpy="1.570796 0.0 1.570796" />
   </joint>
   <xacro:ur5_robot prefix="" joint_limited="true"

Commit message: fixing frames and positions

File: urdf/robotic_arm_inspector.urdf.xacro (robot description, xacro)
@@ -11,5 +11,5 @@
     <parent link="world" />
     <child link = "cart" />
-    <origin xyz="0.0 0.0 1.0" rpy="0.0 0.0 0.0" />
+    <origin xyz="0.0 0.0 1.0"/>
   </joint>
   <link name = "cart"/>
@@ -17,5 +17,5 @@
     <parent link="cart" />
     <child link = "base_link" />
-    <origin xyz="0.0 0.7 0.0" rpy="1.570796 0.0 1.570796" />
+    <origin xyz="0.0 1.5 0.0"  rpy="1.570796 0.0 1.570796"/>
   </joint>
   <xacro:ur5_robot prefix="" joint_limited="true"
