Commit message: Update kinect.urdf.xacro
updated with the used local version in which the collision was enabled and the kinect moved a bit forward to avoid always self collision

File: urdf/used_sensors/kinect.urdf.xacro (robot description, xacro)
@@ -45,10 +45,10 @@
 				</geometry>
 			</visual>
-			<!-- <collision>
+			<collision>
 				<origin xyz="0.0 0.0 0.0" rpy="0 0 0"/>
 				<geometry>
 					<box size="0.07271 0.27794 0.073"/>
 				</geometry>
-			</collision> -->
+			</collision>
 			<inertial>
 				<mass value="0.001" />
